Commit message: Finshing Jaguar class and starting with the arm

File: src/mini_jaguar_pkg/urdf/robot_parameters.xacro (robot description, xacro)
@@ -2,18 +2,18 @@
 <robot xmlns:xacro="http://www.ros.org/wiki/xacro">
   <xacro:property name="link_00_name" value="base_link" />
-  <xacro:property name="link_01_name" value="link_01" />
-  <xacro:property name="link_02_name" value="link_02" />
-  <xacro:property name="link_03_name" value="link_03" />
-  <xacro:property name="link_04_name" value="link_04" />
-  <xacro:property name="link_05_name" value="link_05" />
-  <xacro:property name="link_06_name" value="link_06" />
-  <xacro:property name="link_07_name" value="link_07" />
-  <xacro:property name="link_08_name" value="link_08" />
-  <xacro:property name="link_09_name" value="link_09" />
-  <xacro:property name="link_10_name" value="link_10" />
-  <xacro:property name="link_11_name" value="link_11" />
-  <xacro:property name="link_12_name" value="link_12" />
-  <xacro:property name="link_13_name" value="link_13" />
-  <xacro:property name="link_14_name" value="link_14" />
-  <xacro:property name="link_15_name" value="link_15" />
+  <xacro:property name="link_01_name" value="base_arm" />
+  <xacro:property name="link_02_name" value="wheel_front_left" />
+  <xacro:property name="link_03_name" value="wheel_front_right" />
+  <xacro:property name="link_04_name" value="wheel_back_right" />
+  <xacro:property name="link_05_name" value="wheel_back_left" />
+  <xacro:property name="link_06_name" value="arm_1" />
+  <xacro:property name="link_07_name" value="arm_2" />
+  <xacro:property name="link_08_name" value="arm_3" />
+  <xacro:property name="link_09_name" value="arm_4" />
+  <xacro:property name="link_10_name" value="griper_1" />
+  <xacro:property name="link_11_name" value="griper_2" />
+  <xacro:property name="link_12_name" value="fliper_front_left" />
+  <xacro:property name="link_13_name" value="fliper_back_left" />
+  <xacro:property name="link_14_name" value="fliper_front_right" />
+  <xacro:property name="link_15_name" value="fliper_back_right" />
 </robot>
