Commit message: adding parts folder

File: src/mini_jaguar_pkg/parts/arm.xacro (robot description, xacro)
@@ -29,9 +29,9 @@
   <m_joint name="${link_06_name}__${link_07_name}" type="revolute"
            axis_xyz="0 1 0"
-           origin_rpy="3.14 3.14 0" origin_xyz="0.44 0 -0.035"
+           origin_rpy="3.14 3.14 0" origin_xyz="0.44 0 -0.015"
            parent="${link_06_name}" child="${link_07_name}"
            limit_e="1000" limit_l="0" limit_u="3.14" limit_v="0.5" />
   <m_link_mesh name="${link_07_name}"
-              origin_rpy="0 0 0" origin_xyz="0 -0.0145 -0.0145"
+              origin_rpy="0 0 0" origin_xyz="0 -0.0145 -0.03"
               mass="157.633"
               ixx="13.235" ixy="0" ixz="0"
@@ -40,3 +40,52 @@
               meshfile="package://mini_jaguar_pkg/meshes/arm.stl"
               meshscale="0.004 0.0029 0.003" />
+  <m_joint name="${link_07_name}__${link_08_name}" type="revolute"
+           axis_xyz="0 1 0"
+           origin_rpy="0 0 0" origin_xyz="0.43 0.025 -0.0145"
+           parent="${link_07_name}" child="${link_08_name}"
+           limit_e="1000" limit_l="-1" limit_u="3.14" limit_v="0.5" />
+  <m_link_mesh name="${link_08_name}"
+              origin_rpy="0 0 0" origin_xyz="-0.15  -0.0145 -0.0145"
+              mass="157.633"
+              ixx="13.235" ixy="0" ixz="0"
+              iyy="13.235" iyz="0"
+              izz="9.655"
+              meshfile="package://mini_jaguar_pkg/meshes/arm.stl"
+              meshscale="0.0025 0.0029 0.003" />
+  <m_joint name="${link_08_name}__${link_09_name}" type="revolute"
+           axis_xyz="0 0 1"
+           origin_rpy="0 1.57079 0" origin_xyz="0.13 0 0"
+           parent="${link_08_name}" child="${link_09_name}"
+           limit_e="1000" limit_l="0" limit_u="3.14" limit_v="0.5" />
+  <m_link_cylinder name="${link_09_name}"
+              origin_rpy="0 0 0" origin_xyz="0 0 0"
+              mass="157.633"
+              ixx="13.235" ixy="0" ixz="0"
+              iyy="13.235" iyz="0"
+              izz="9.655"
+              radius='.015' length='0.01'/>
+  <m_joint name="${link_09_name}__${link_10_name}" type="revolute"
+           axis_xyz="1 0 0"
+           origin_rpy="0 0 0" origin_xyz="0 0.018 0.0"
+           parent="${link_09_name}" child="${link_10_name}"
+           limit_e="1000" limit_l="0" limit_u="0.32" limit_v="0.5" />
+   <m_link_box name="${link_10_name}"
+              origin_rpy="0 0 0" origin_xyz="0 0 0.02"
+              mass="157.633"
+              ixx="13.235" ixy="0" ixz="0"
+              iyy="13.235" iyz="0"
+              izz="9.655"
+              size='0.02 0.005 0.05'/>
+  <m_joint name="${link_09_name}__${link_11_name}" type="revolute"
+           axis_xyz="1 0 0"
+           origin_rpy="0 0 3.14" origin_xyz="0 -0.018 0.0"
+           parent="${link_09_name}" child="${link_11_name}"
+           limit_e="1000" limit_l="0" limit_u="0.32" limit_v="0.5" />
+   <m_link_box name="${link_11_name}"
+              origin_rpy="0 0 0" origin_xyz="0 0 0.02"
+              mass="157.633"
+              ixx="13.235" ixy="0" ixz="0"
+              iyy="13.235" iyz="0"
+              izz="9.655"
+              size='0.02 0.005 0.05'/>
 </robot>

File: src/mini_jaguar_pkg/urdf/mini.xacro (robot description, xacro)
@@ -6,4 +6,5 @@
   <xacro:include filename="$(find mini_jaguar_pkg)/parts/wheels.xacro" />
   <xacro:include filename="$(find mini_jaguar_pkg)/parts/arm.xacro" />
+  <xacro:include filename="$(find mini_jaguar_pkg)/parts/fins.xacro" />
   <!-- END - Include -->
   <link name='chassis'>

File: src/mini_jaguar_pkg/urdf/robot_parameters.xacro (robot description, xacro)
@@ -12,3 +12,8 @@
   <xacro:property name="link_09_name" value="link_09" />
   <xacro:property name="link_10_name" value="link_10" />
+  <xacro:property name="link_11_name" value="link_11" />
+  <xacro:property name="link_12_name" value="link_12" />
+  <xacro:property name="link_13_name" value="link_13" />
+  <xacro:property name="link_14_name" value="link_14" />
+  <xacro:property name="link_15_name" value="link_15" />
 </robot>

Commit message: Changing joints naming

File: src/mini_jaguar_pkg/parts/arm.xacro (robot description, xacro)
@@ -1,8 +1,8 @@
 <?xml version="1.0" ?>
 <robot xmlns:xacro="http://www.ros.org/wiki/xacro">
-  <m_joint name="chassis__${link_01_name}" type="revolute"
+  <m_joint name="${link_00_name}__${link_01_name}" type="revolute"
            axis_xyz="0 0 1"
            origin_rpy="0 0 0" origin_xyz="0.2 0 0.05"
-           parent="chassis" child="link_01"
+           parent="${link_00_name}" child="${link_01_name}"
            limit_e="1000" limit_l="-3.14" limit_u="3.14" limit_v="0.5" />
   <m_link_mesh name="${link_01_name}"

File: src/mini_jaguar_pkg/parts/fins.xacro (robot description, xacro)
@@ -1,8 +1,8 @@
 <?xml version="1.0" ?>
 <robot xmlns:xacro="http://www.ros.org/wiki/xacro">
-  <m_joint name="chassis__${link_12_name}" type="revolute"
+  <m_joint name="${link_00_name}__${link_12_name}" type="revolute"
            axis_xyz="0 1 0"
            origin_rpy="0 0 3.14" origin_xyz="0.27 0.24 0"
-           parent="chassis" child="${link_12_name}"
+           parent="${link_00_name}" child="${link_12_name}"
            limit_e="1000" limit_l="-3.14" limit_u="3.14" limit_v="0.5" />
   <m_link_mesh name="${link_12_name}"
@@ -14,8 +14,8 @@
               meshfile="package://mini_jaguar_pkg/meshes/arm.stl"
               meshscale="0.0025 0.0029 0.003" />
-  <m_joint name="chassis__${link_13_name}" type="revolute"
+  <m_joint name="${link_00_name}__${link_13_name}" type="revolute"
            axis_xyz="0 1 0"
            origin_rpy="0 0 3.14" origin_xyz="-0.27 0.24 0"
-           parent="chassis" child="${link_13_name}"
+           parent="${link_00_name}" child="${link_13_name}"
            limit_e="1000" limit_l="-3.14" limit_u="3.14" limit_v="0.5" />
   <m_link_mesh name="${link_13_name}"
@@ -27,8 +27,8 @@
               meshfile="package://mini_jaguar_pkg/meshes/arm.stl"
               meshscale="0.0025 0.0029 0.003" />
-  <m_joint name="chassis__${link_14_name}" type="revolute"
+  <m_joint name="${link_00_name}__${link_14_name}" type="revolute"
            axis_xyz="0 1 0"
            origin_rpy="0 0 3.14" origin_xyz="0.27 -0.3 0"
-           parent="chassis" child="${link_14_name}"
+           parent="${link_00_name}" child="${link_14_name}"
            limit_e="1000" limit_l="-3.14" limit_u="3.14" limit_v="0.5" />
   <m_link_mesh name="${link_14_name}"
@@ -40,8 +40,8 @@
               meshfile="package://mini_jaguar_pkg/meshes/arm.stl"
               meshscale="0.0025 0.0029 0.003" />
-  <m_joint name="chassis__${link_15_name}" type="revolute"
+  <m_joint name="${link_00_name}__${link_15_name}" type="revolute"
            axis_xyz="0 1 0"
            origin_rpy="0 0 3.14" origin_xyz="-0.27 -0.30 0"
-           parent="chassis" child="${link_15_name}"
+           parent="${link_00_name}" child="${link_15_name}"
            limit_e="1000" limit_l="-3.14" limit_u="3.14" limit_v="0.5" />
   <m_link_mesh name="${link_15_name}"

File: src/mini_jaguar_pkg/parts/wheels.xacro (robot description, xacro)
@@ -1,8 +1,8 @@
 <?xml version="1.0" ?>
 <robot xmlns:xacro="http://www.ros.org/wiki/xacro">
-   <m_joint name="chassis__${link_02_name}" type="revolute"
+   <m_joint name="${link_00_name}__${link_02_name}" type="revolute"
            axis_xyz="0 1 0"
            origin_rpy="0 0 0" origin_xyz="0.27 0.23 0"
-           parent="chassis" child="link_02"
+           parent="${link_00_name}" child="${link_02_name}"
            limit_e="1000" limit_l="-3.14" limit_u="3.14" limit_v="0.5" />
   <m_link_mesh name="${link_02_name}"
@@ -14,8 +14,8 @@
               meshfile="package://mini_jaguar_pkg/meshes/tyre.dae"
               meshscale="1.7 1.7 1.7" />
-    <m_joint name="chassis__${link_03_name}" type="revolute"
+    <m_joint name="${link_00_name}__${link_03_name}" type="revolute"
            axis_xyz="0 1 0"
            origin_rpy="0 0 0" origin_xyz="0.27 -0.23 0"
-           parent="chassis" child="link_03"
+           parent="${link_00_name}" child="${link_03_name}"
            limit_e="1000" limit_l="-3.14" limit_u="3.14" limit_v="0.5" />
   <m_link_mesh name="${link_03_name}"
@@ -27,8 +27,8 @@
               meshfile="package://mini_jaguar_pkg/meshes/tyre.dae"
               meshscale="1.7 1.7 1.7" />
-    <m_joint name="chassis__${link_04_name}" type="revolute"
+    <m_joint name="${link_00_name}__${link_04_name}" type="revolute"
            axis_xyz="0 1 0"
            origin_rpy="0 0 0" origin_xyz="-0.27 -0.23 0"
-           parent="chassis" child="link_04"
+           parent="${link_00_name}" child="${link_04_name}"
            limit_e="1000" limit_l="-3.14" limit_u="3.14" limit_v="0.5" />
   <m_link_mesh name="${link_04_name}"
@@ -40,8 +40,8 @@
               meshfile="package://mini_jaguar_pkg/meshes/tyre.dae"
               meshscale="1.7 1.7 1.7" />
-      <m_joint name="chassis__${link_05_name}" type="revolute"
+      <m_joint name="${link_00_name}__${link_05_name}" type="revolute"
            axis_xyz="0 1 0"
            origin_rpy="0 0 0" origin_xyz="-0.27 0.23 0"
-           parent="chassis" child="link_05"
+           parent="${link_00_name}" child="${link_05_name}"
            limit_e="1000" limit_l="-3.14" limit_u="3.14" limit_v="0.5" />
   <m_link_mesh name="${link_05_name}"

File: src/mini_jaguar_pkg/urdf/mini.xacro (robot description, xacro)
@@ -8,5 +8,5 @@
   <xacro:include filename="$(find mini_jaguar_pkg)/parts/fins.xacro" />
   <!-- END - Include -->
-  <link name='chassis'>
+  <link name='${link_00_name}'>
     <pose>0 0 0.1 0 0 0</pose>
     <inertial>
