Commit message: adding the nav stack

File: src/mini_jaguar_pkg/parts/arm.xacro (robot description, xacro)
@@ -3,7 +3,7 @@
   <m_joint name="${link_00_name}__${link_01_name}" type="revolute"
            axis_xyz="0 0 1"
-           origin_rpy="0 0 0" origin_xyz="0.2 0 0.05"
+           origin_rpy="0 0 0" origin_xyz="0.13 0 0.27"
            parent="${link_00_name}" child="${link_01_name}"
-           limit_e="1000" limit_l="-3.14" limit_u="3.14" limit_v="0.5" />
+           limit_e="1000" limit_l="-1.5708" limit_u="1.5708" limit_v="0.5" />
   <m_link_mesh name="${link_01_name}"
               origin_rpy="0 0 0" origin_xyz="0 0 0"
@@ -12,51 +12,12 @@
               iyy="13.235" iyz="0"
               izz="9.655"
-              meshfile="package://mini_jaguar_pkg/meshes/armBase.stl"
-              meshscale="0.0003 0.0003 0.0003" />
+              meshfile="package://mini_jaguar_pkg/meshes/Arm_Base_scaled.dae"
+              meshscale="1 1 1" />
   <m_joint name="${link_01_name}__${link_06_name}" type="revolute"
            axis_xyz="0 1 0"
-           origin_rpy="0 3.14 0" origin_xyz="0 0 0.13"
+           origin_rpy="0 0.05 0" origin_xyz="0.1 0.045 0.12"
            parent="${link_01_name}" child="${link_06_name}"
            limit_e="1000" limit_l="0" limit_u="3.14" limit_v="0.5" />
   <m_link_mesh name="${link_06_name}"
-              origin_rpy="0 0 0" origin_xyz="0 -0.0145 -0.0145"
-              mass="157.633"
-              ixx="13.235" ixy="0" ixz="0"
-              iyy="13.235" iyz="0"
-              izz="9.655"
-              meshfile="package://mini_jaguar_pkg/meshes/arm.stl"
-              meshscale="0.004 0.0029 0.003" />
-  <m_joint name="${link_06_name}__${link_07_name}" type="revolute"
-           axis_xyz="0 1 0"
-           origin_rpy="3.14 3.14 0" origin_xyz="0.44 0 -0.015"
-           parent="${link_06_name}" child="${link_07_name}"
-           limit_e="1000" limit_l="0" limit_u="3.14" limit_v="0.5" />
-  <m_link_mesh name="${link_07_name}"
-              origin_rpy="0 0 0" origin_xyz="0 -0.0145 -0.03"
-              mass="157.633"
-              ixx="13.235" ixy="0" ixz="0"
-              iyy="13.235" iyz="0"
-              izz="9.655"
-              meshfile="package://mini_jaguar_pkg/meshes/arm.stl"
-              meshscale="0.004 0.0029 0.003" />
-  <m_joint name="${link_07_name}__${link_08_name}" type="revolute"
-           axis_xyz="0 1 0"
-           origin_rpy="0 0 0" origin_xyz="0.43 0.025 -0.0145"
-           parent="${link_07_name}" child="${link_08_name}"
-           limit_e="1000" limit_l="-1" limit_u="3.14" limit_v="0.5" />
-  <m_link_mesh name="${link_08_name}"
-              origin_rpy="0 0 0" origin_xyz="-0.15  -0.0145 -0.0145"
-              mass="157.633"
-              ixx="13.235" ixy="0" ixz="0"
-              iyy="13.235" iyz="0"
-              izz="9.655"
-              meshfile="package://mini_jaguar_pkg/meshes/arm.stl"
-              meshscale="0.0025 0.0029 0.003" />
-  <m_joint name="${link_08_name}__${link_09_name}" type="revolute"
-           axis_xyz="0 0 1"
-           origin_rpy="0 1.57079 0" origin_xyz="0.13 0 0"
-           parent="${link_08_name}" child="${link_09_name}"
-           limit_e="1000" limit_l="0" limit_u="3.14" limit_v="0.5" />
-  <m_link_cylinder name="${link_09_name}"
               origin_rpy="0 0 0" origin_xyz="0 0 0"
               mass="157.633"
@@ -64,5 +25,46 @@
               iyy="13.235" iyz="0"
               izz="9.655"
-              radius='.015' length='0.01'/>
+              meshfile="package://mini_jaguar_pkg/meshes/Arm_1_scaled.dae"
+              meshscale="1 1 1" />
+  <m_joint name="${link_06_name}__${link_07_name}" type="revolute"
+           axis_xyz="0 1 0"
+           origin_rpy="0 0 3.14" origin_xyz="-0.46 -0.1335 0"
+           parent="${link_06_name}" child="${link_07_name}"
+           limit_e="1000" limit_l="0" limit_u="3.14" limit_v="0.5" />
+  <m_link_mesh name="${link_07_name}"
+              origin_rpy="3.14 3.14 0" origin_xyz="0 0 0"
+              mass="157.633"
+              ixx="13.235" ixy="0" ixz="0"
+              iyy="13.235" iyz="0"
+              izz="9.655"
+              meshfile="package://mini_jaguar_pkg/meshes/Arm_2_scaled.dae"
+              meshscale="1 1 1" />
+  <m_joint name="${link_07_name}__${link_08_name}" type="revolute"
+           axis_xyz="0 1 0"
+           origin_rpy="0 0 0" origin_xyz="-0.43 -0.036 0.14"
+           parent="${link_07_name}" child="${link_08_name}"
+           limit_e="1000" limit_l="-1" limit_u="3.14" limit_v="0.5" />
+  <m_link_mesh name="${link_08_name}"
+              origin_rpy="0 0 3.14" origin_xyz="0 0 0"
+              mass="157.633"
+              ixx="13.235" ixy="0" ixz="0"
+              iyy="13.235" iyz="0"
+              izz="9.655"
+              meshfile="package://mini_jaguar_pkg/meshes/Arm_3_scaled.dae"
+              meshscale="1 1 1" />
+  <m_joint name="${link_08_name}__${link_09_name}" type="revolute"
+           axis_xyz="1 0 0"
+           origin_rpy="0 -0.18 3.14" origin_xyz="-0.08 -0.0346 0.014"
+           parent="${link_08_name}" child="${link_09_name}"
+           limit_e="1000" limit_l="-3.14" limit_u="3.14" limit_v="0.5" />
+  <m_link_mesh name="${link_09_name}"
+              origin_rpy="0 0.17 0" origin_xyz="0 0 0"
+              mass="157.633"
+              ixx="13.235" ixy="0" ixz="0"
+              iyy="13.235" iyz="0"
+              izz="9.655"
+              meshfile="package://mini_jaguar_pkg/meshes/Arm_4_scaled.dae"
+              meshscale="1 1 1" />
+<!--
   <m_joint name="${link_09_name}__${link_10_name}" type="revolute"
            axis_xyz="1 0 0"
@@ -88,4 +90,4 @@
               iyy="13.235" iyz="0"
               izz="9.655"
-              size='0.02 0.005 0.05'/>
+              size='0.02 0.005 0.05'/>   -->
 </robot>

File: src/mini_jaguar_pkg/parts/fins.xacro (robot description, xacro)
@@ -3,53 +3,53 @@
   <m_joint name="${link_00_name}__${link_12_name}" type="revolute"
            axis_xyz="0 1 0"
-           origin_rpy="0 0 3.14" origin_xyz="0.27 0.24 0"
+           origin_rpy="0 3.14 0" origin_xyz="0.24 0.28 0.13"
            parent="${link_00_name}" child="${link_12_name}"
            limit_e="1000" limit_l="-3.14" limit_u="3.14" limit_v="0.5" />
   <m_link_mesh name="${link_12_name}"
-              origin_rpy="0 0 3.14" origin_xyz="0  -0.0145 -0.0145"
+              origin_rpy="0 0 3.14" origin_xyz="0  0 0"
               mass="157.633"
               ixx="13.235" ixy="0" ixz="0"
               iyy="13.235" iyz="0"
               izz="9.655"
-              meshfile="package://mini_jaguar_pkg/meshes/arm.stl"
-              meshscale="0.0025 0.0029 0.003" />
+              meshfile="package://mini_jaguar_pkg/meshes/flipper.dae"
+              meshscale="1 1 1" />
   <m_joint name="${link_00_name}__${link_13_name}" type="revolute"
            axis_xyz="0 1 0"
-           origin_rpy="0 0 3.14" origin_xyz="-0.27 0.24 0"
+           origin_rpy="0 0 0" origin_xyz="-0.24 0.28 0.13"
            parent="${link_00_name}" child="${link_13_name}"
            limit_e="1000" limit_l="-3.14" limit_u="3.14" limit_v="0.5" />
   <m_link_mesh name="${link_13_name}"
-              origin_rpy="0 0 3.14" origin_xyz="0  -0.0145 -0.0145"
+              origin_rpy="0 0 3.14" origin_xyz="0 0 0"
               mass="157.633"
               ixx="13.235" ixy="0" ixz="0"
               iyy="13.235" iyz="0"
               izz="9.655"
-              meshfile="package://mini_jaguar_pkg/meshes/arm.stl"
-              meshscale="0.0025 0.0029 0.003" />
+              meshfile="package://mini_jaguar_pkg/meshes/flipper.dae"
+              meshscale="1 1 1" />
   <m_joint name="${link_00_name}__${link_14_name}" type="revolute"
            axis_xyz="0 1 0"
-           origin_rpy="0 0 3.14" origin_xyz="0.27 -0.3 0"
+           origin_rpy="0 3.14 0" origin_xyz="-0.24 -0.28 0.13"
            parent="${link_00_name}" child="${link_14_name}"
            limit_e="1000" limit_l="-3.14" limit_u="3.14" limit_v="0.5" />
   <m_link_mesh name="${link_14_name}"
-              origin_rpy="0 0 3.14" origin_xyz="0  -0.0145 -0.0145"
+              origin_rpy="0 0 0" origin_xyz="0 0 0"
               mass="157.633"
               ixx="13.235" ixy="0" ixz="0"
               iyy="13.235" iyz="0"
               izz="9.655"
-              meshfile="package://mini_jaguar_pkg/meshes/arm.stl"
-              meshscale="0.0025 0.0029 0.003" />
+              meshfile="package://mini_jaguar_pkg/meshes/flipper.dae"
+              meshscale="1 1 1" />
   <m_joint name="${link_00_name}__${link_15_name}" type="revolute"
            axis_xyz="0 1 0"
-           origin_rpy="0 0 3.14" origin_xyz="-0.27 -0.30 0"
+           origin_rpy="0 0 3.14" origin_xyz="0.24 -0.28 0.13"
            parent="${link_00_name}" child="${link_15_name}"
            limit_e="1000" limit_l="-3.14" limit_u="3.14" limit_v="0.5" />
   <m_link_mesh name="${link_15_name}"
-              origin_rpy="0 0 3.14" origin_xyz="0  -0.0145 -0.0145"
+              origin_rpy="0 0 3.14" origin_xyz="0 0 0"
               mass="157.633"
               ixx="13.235" ixy="0" ixz="0"
               iyy="13.235" iyz="0"
               izz="9.655"
-              meshfile="package://mini_jaguar_pkg/meshes/arm.stl"
-              meshscale="0.0025 0.0029 0.003" />
+              meshfile="package://mini_jaguar_pkg/meshes/flipper.dae"
+              meshscale="1 1 1" />
 </robot>

File: src/mini_jaguar_pkg/parts/wheels.xacro (robot description, xacro)
@@ -3,7 +3,7 @@
    <m_joint name="${link_00_name}__${link_02_name}" type="revolute"
            axis_xyz="0 1 0"
-           origin_rpy="0 0 0" origin_xyz="0.27 0.23 0"
+           origin_rpy="0 0 0" origin_xyz="0 0.206 0.13"
            parent="${link_00_name}" child="${link_02_name}"
-           limit_e="1000" limit_l="-3.14" limit_u="3.14" limit_v="0.5" />
+           limit_e="1000" limit_l="0" limit_u="0" limit_v="0" />
   <m_link_mesh name="${link_02_name}"
               origin_rpy="0 0 0" origin_xyz="0 0 0"
@@ -12,19 +12,22 @@
               iyy="13.235" iyz="0"
               izz="9.655"
-              meshfile="package://mini_jaguar_pkg/meshes/tyre.dae"
-              meshscale="1.7 1.7 1.7" />
+              meshfile="package://mini_jaguar_pkg/meshes/track.dae"
+              meshscale="1 1 1"/>
     <m_joint name="${link_00_name}__${link_03_name}" type="revolute"
            axis_xyz="0 1 0"
-           origin_rpy="0 0 0" origin_xyz="0.27 -0.23 0"
+           origin_rpy="0 0 3.14" origin_xyz="0 -0.206 0.13"
            parent="${link_00_name}" child="${link_03_name}"
-           limit_e="1000" limit_l="-3.14" limit_u="3.14" limit_v="0.5" />
-  <m_link_mesh name="${link_03_name}"
-              origin_rpy="0 0 0" origin_xyz="0 0 0"
-              mass="157.633"
-              ixx="13.235" ixy="0" ixz="0"
-              iyy="13.235" iyz="0"
-              izz="9.655"
-              meshfile="package://mini_jaguar_pkg/meshes/tyre.dae"
-              meshscale="1.7 1.7 1.7" />
+           limit_e="1000" limit_l="0" limit_u="0" limit_v="0"
+           />
+           <!-- limit_e="1000" limit_l="-3.14" limit_u="3.14" limit_v="0.5"  -->
+    <m_link_mesh name="${link_03_name}"
+                origin_rpy="0 0 0" origin_xyz="0 0 0"
+                mass="157.633"
+                ixx="13.235" ixy="0" ixz="0"
+                iyy="13.235" iyz="0"
+                izz="9.655"
+                meshfile="package://mini_jaguar_pkg/meshes/track.dae"
+                meshscale="1 1 1" />
+ <!--
     <m_joint name="${link_00_name}__${link_04_name}" type="revolute"
            axis_xyz="0 1 0"
@@ -52,4 +55,4 @@
               izz="9.655"
               meshfile="package://mini_jaguar_pkg/meshes/tyre.dae"
-              meshscale="1.7 1.7 1.7" />
+              meshscale="1.7 1.7 1.7" />  -->
 </robot>

File: src/mini_jaguar_pkg/urdf/mini.xacro (robot description, xacro)
@@ -5,12 +5,20 @@
   <xacro:include filename="$(find mini_jaguar_pkg)/urdf/links_joints.xacro" />
   <xacro:include filename="$(find mini_jaguar_pkg)/parts/wheels.xacro" />
-  <xacro:include filename="$(find mini_jaguar_pkg)/parts/arm.xacro" />
   <xacro:include filename="$(find mini_jaguar_pkg)/parts/fins.xacro" />
+   <xacro:include filename="$(find mini_jaguar_pkg)/parts/arm.xacro" />
   <!-- END - Include -->
-  <link name='${link_00_name}'>
+  <m_link_mesh name="${link_00_name}"
+              origin_rpy="0 0 0" origin_xyz="0 0 0.19"
+              mass="157.633"
+              ixx="13.235" ixy="0" ixz="0"
+              iyy="13.235" iyz="0"
+              izz="9.655"
+              meshfile="package://mini_jaguar_pkg/meshes/jaguar_base.dae"
+              meshscale="1 1 1" />
+  <!-- <link name='${link_00_name}'>
     <pose>0 0 0.1 0 0 0</pose>
     <inertial>
       <mass value="15.0"/>
-      <origin xyz="0.0 0 0.1" rpy=" 0 0 0"/>
+      <origin xyz="0.0 0 0.1" rpy="0 0 0"/>
       <inertia
           ixx="0.1" ixy="0" ixz="0"
@@ -30,4 +38,4 @@
       </geometry>
     </visual>
-  </link>
+  </link>     -->
 </robot>

File: src/mini_jaguar_pkg/urdf/robot_parameters.xacro (robot description, xacro)
@@ -3,8 +3,8 @@
   <xacro:property name="link_00_name" value="base_link" />
   <xacro:property name="link_01_name" value="base_arm" />
-  <xacro:property name="link_02_name" value="wheel_front_left" />
-  <xacro:property name="link_03_name" value="wheel_front_right" />
-  <xacro:property name="link_04_name" value="wheel_back_right" />
-  <xacro:property name="link_05_name" value="wheel_back_left" />
+  <xacro:property name="link_02_name" value="wheel_left" />
+  <xacro:property name="link_03_name" value="wheel_right" />
+  <!-- <xacro:property name="link_04_name" value="wheel_back_right" />
+  <xacro:property name="link_05_name" value="wheel_back_left" /> -->
   <xacro:property name="link_06_name" value="arm_1" />
   <xacro:property name="link_07_name" value="arm_2" />
