Commit message: Move workspace

File: src/mini_jaguar_pkg/parts/arm.xacro (robot description, xacro)
@@ -12,5 +12,5 @@
               iyy="13.235" iyz="0"
               izz="9.655"
-              meshfile="package://mini_jaguar_pkg/meshes/Arm_Base_scaled.dae"
+              meshfile="package://mini_jaguar_pkg/meshes/jaguar/Arm_Base_scaled.dae"
               meshscale="1 1 1" />
   <m_joint name="${link_01_name}__${link_06_name}" type="revolute"
@@ -25,5 +25,5 @@
               iyy="13.235" iyz="0"
               izz="9.655"
-              meshfile="package://mini_jaguar_pkg/meshes/Arm_1_scaled.dae"
+              meshfile="package://mini_jaguar_pkg/meshes/jaguar/Arm_1_scaled.dae"
               meshscale="1 0.95 1" />
   <m_joint name="${link_06_name}__${link_07_name}" type="revolute"
@@ -38,5 +38,5 @@
               iyy="13.235" iyz="0"
               izz="9.655"
-              meshfile="package://mini_jaguar_pkg/meshes/Arm_2_scaled.dae"
+              meshfile="package://mini_jaguar_pkg/meshes/jaguar/Arm_2_scaled.dae"
               meshscale="1 1 1" />
   <m_joint name="${link_07_name}__${link_08_name}" type="revolute"
@@ -44,5 +44,5 @@
            origin_rpy="0 0 0" origin_xyz="-0.43 -0.044 0.14"
            parent="${link_07_name}" child="${link_08_name}"
-           limit_e="1000" limit_l="-3.14" limit_u="3.14" limit_v="0.5" />
+           limit_e="1000" limit_l="0" limit_u="0" limit_v="0" />
   <m_link_mesh name="${link_08_name}"
               origin_rpy="0 0 3.14" origin_xyz="0 0 0"
@@ -51,5 +51,5 @@
               iyy="13.235" iyz="0"
               izz="9.655"
-              meshfile="package://mini_jaguar_pkg/meshes/Arm_3_scaled.dae"
+              meshfile="package://mini_jaguar_pkg/meshes/jaguar/Arm_3_scaled.dae"
               meshscale="1 1 1" />
   <m_joint name="${link_08_name}__${link_09_name}" type="revolute"
@@ -64,5 +64,5 @@
               iyy="13.235" iyz="0"
               izz="9.655"
-              meshfile="package://mini_jaguar_pkg/meshes/Arm_4_scaled.dae"
+              meshfile="package://mini_jaguar_pkg/meshes/jaguar/Arm_4_scaled.dae"
               meshscale="1 1.1 1" />
 </robot>

File: src/mini_jaguar_pkg/parts/fins.xacro (robot description, xacro)
@@ -25,5 +25,5 @@
               iyy="13.235" iyz="0"
               izz="9.655"
-              meshfile="package://mini_jaguar_pkg/meshes/flipper.dae"
+              meshfile="package://mini_jaguar_pkg/meshes/jaguar/flipper.dae"
               meshscale="1 1 1" />
    <m_joint name="${link_00_name}__${link_13_name}" type="revolute"
@@ -38,5 +38,5 @@
               iyy="13.235" iyz="0"
               izz="9.655"
-              meshfile="package://mini_jaguar_pkg/meshes/flipper.dae"
+              meshfile="package://mini_jaguar_pkg/meshes/jaguar/flipper.dae"
               meshscale="1 1 1" />
    <m_joint name="${link_00_name}__${link_14_name}" type="revolute"
@@ -51,5 +51,5 @@
               iyy="13.235" iyz="0"
               izz="9.655"
-              meshfile="package://mini_jaguar_pkg/meshes/flipper.dae"
+              meshfile="package://mini_jaguar_pkg/meshes/jaguar/flipper.dae"
               meshscale="1 1 1" />
   <m_joint name="${link_00_name}__${link_15_name}" type="revolute"
@@ -64,5 +64,5 @@
               iyy="13.235" iyz="0"
               izz="9.655"
-              meshfile="package://mini_jaguar_pkg/meshes/flipper.dae"
+              meshfile="package://mini_jaguar_pkg/meshes/jaguar/flipper.dae"
               meshscale="1 1 1" />
 </robot>

File: src/mini_jaguar_pkg/parts/wheels.xacro (robot description, xacro)
@@ -1,58 +1,59 @@
 <?xml version="1.0" ?>
 <robot xmlns:xacro="http://www.ros.org/wiki/xacro">
-   <m_joint name="${link_00_name}__${link_02_name}" type="revolute"
+<xacro:property name="meshscaleX" value="2.5" />
+<xacro:property name="meshscaleY" value="2.5" />
+<xacro:property name="meshscaleZ" value="2.5" />
+  <m_joint name="${link_00_name}__${link_02_name}" type="continuous"
            axis_xyz="0 1 0"
-           origin_rpy="0 0 0" origin_xyz="0 0.215 0.13"
+           origin_rpy="0 0 0" origin_xyz="0.27 0.24 0.12"
            parent="${link_00_name}" child="${link_02_name}"
-           limit_e="1000" limit_l="0" limit_u="0" limit_v="0" />
+            limit_e="1000" limit_l="-3.14" limit_u="3.14" limit_v="0.5"
+              />
   <m_link_mesh name="${link_02_name}"
               origin_rpy="0 0 0" origin_xyz="0 0 0"
-              mass="157.633"
+              mass="15.633"
               ixx="13.235" ixy="0" ixz="0"
               iyy="13.235" iyz="0"
               izz="9.655"
-              meshfile="package://mini_jaguar_pkg/meshes/track.dae"
-              meshscale="1 1 1"/>
-    <m_joint name="${link_00_name}__${link_03_name}" type="revolute"
+              meshfile="package://mini_jaguar_pkg/meshes/jaguar/wheel.dae"
+              meshscale="${meshscaleX} ${meshscaleY} ${meshscaleZ}"/>
+    <m_joint name="${link_00_name}__${link_03_name}" type="continuous"
            axis_xyz="0 1 0"
-           origin_rpy="0 0 3.14" origin_xyz="0 -0.215 0.13"
+           origin_rpy="0 0 0" origin_xyz="0.27 -0.24 0.12"
            parent="${link_00_name}" child="${link_03_name}"
-           limit_e="1000" limit_l="0" limit_u="0" limit_v="0"
-           />
-           <!-- limit_e="1000" limit_l="-3.14" limit_u="3.14" limit_v="0.5"  -->
+       limit_e="1000" limit_l="-3.14" limit_u="3.14" limit_v="0.5" />
     <m_link_mesh name="${link_03_name}"
                 origin_rpy="0 0 0" origin_xyz="0 0 0"
-                mass="157.633"
+                mass="15.633"
                 ixx="13.235" ixy="0" ixz="0"
                 iyy="13.235" iyz="0"
                 izz="9.655"
-                meshfile="package://mini_jaguar_pkg/meshes/track.dae"
-                meshscale="1 1 1" />
- <!--
-    <m_joint name="${link_00_name}__${link_04_name}" type="revolute"
+                meshfile="package://mini_jaguar_pkg/meshes/jaguar/wheel.dae"
+                meshscale="{meshscaleX} ${meshscaleY} ${meshscaleZ}" />
+    <m_joint name="${link_00_name}__${link_04_name}" type="continuous"
            axis_xyz="0 1 0"
-           origin_rpy="0 0 0" origin_xyz="-0.27 -0.23 0"
+           origin_rpy="0 0 0" origin_xyz="-0.27 -0.24 0.12"
            parent="${link_00_name}" child="${link_04_name}"
            limit_e="1000" limit_l="-3.14" limit_u="3.14" limit_v="0.5" />
   <m_link_mesh name="${link_04_name}"
               origin_rpy="0 0 0" origin_xyz="0 0 0"
-              mass="157.633"
+              mass="15.633"
               ixx="13.235" ixy="0" ixz="0"
               iyy="13.235" iyz="0"
               izz="9.655"
-              meshfile="package://mini_jaguar_pkg/meshes/tyre.dae"
-              meshscale="1.7 1.7 1.7" />
-      <m_joint name="${link_00_name}__${link_05_name}" type="revolute"
+              meshfile="package://mini_jaguar_pkg/meshes/jaguar/wheel.dae"
+              meshscale="{meshscaleX} ${meshscaleY} ${meshscaleZ}" />
+      <m_joint name="${link_00_name}__${link_05_name}" type="continuous"
            axis_xyz="0 1 0"
-           origin_rpy="0 0 0" origin_xyz="-0.27 0.23 0"
+           origin_rpy="0 0 0" origin_xyz="-0.27 0.24 0.12"
            parent="${link_00_name}" child="${link_05_name}"
            limit_e="1000" limit_l="-3.14" limit_u="3.14" limit_v="0.5" />
   <m_link_mesh name="${link_05_name}"
               origin_rpy="0 0 0" origin_xyz="0 0 0"
-              mass="157.633"
+              mass="15.633"
               ixx="13.235" ixy="0" ixz="0"
               iyy="13.235" iyz="0"
               izz="9.655"
-              meshfile="package://mini_jaguar_pkg/meshes/tyre.dae"
-              meshscale="1.7 1.7 1.7" />  -->
+              meshfile="package://mini_jaguar_pkg/meshes/jaguar/wheel.dae"
+              meshscale="{meshscaleX} ${meshscaleY} ${meshscaleZ}" />
 </robot>

File: src/mini_jaguar_pkg/urdf/mini.xacro (robot description, xacro)
@@ -5,24 +5,16 @@
   <xacro:include filename="$(find mini_jaguar_pkg)/urdf/links_joints.xacro" />
   <xacro:include filename="$(find mini_jaguar_pkg)/parts/wheels.xacro" />
+  <xacro:include filename="$(find mini_jaguar_pkg)/parts/arm.xacro" />
   <xacro:include filename="$(find mini_jaguar_pkg)/parts/fins.xacro" />
-  <xacro:include filename="$(find mini_jaguar_pkg)/parts/arm.xacro" />
   <!-- END - Include -->
-  <m_link_mesh name="${link_00_name}"
-              origin_rpy="0 0 0" origin_xyz="0 0 0.19"
-              mass="157.633"
-              ixx="13.235" ixy="0" ixz="0"
-              iyy="13.235" iyz="0"
-              izz="9.655"
-              meshfile="package://mini_jaguar_pkg/meshes/jaguar_base.dae"
-              meshscale="1 1 1"/>
-  <!-- <link name='${link_00_name}'>
+  <link name='${link_00_name}'>
     <pose>0 0 0.1 0 0 0</pose>
     <inertial>
       <mass value="15.0"/>
-      <origin xyz="0.0 0 0.1" rpy="0 0 0"/>
+      <origin xyz="0.0 0 0.1" rpy=" 0 0 0"/>
       <inertia
-          ixx="0.1" ixy="0" ixz="0"
-          iyy="0.1" iyz="0"
-          izz="0.1"
+          ixx="50.1" ixy="0" ixz="0"
+          iyy="013.1" iyz="0"
+          izz="013.1"
       />
     </inertial>
@@ -38,4 +30,4 @@
       </geometry>
     </visual>
-  </link>     -->
+  </link>
 </robot>

File: src/mini_jaguar_pkg/urdf/robot_parameters.xacro (robot description, xacro)
@@ -1,10 +1,11 @@
 <?xml version="1.0" ?>
 <robot xmlns:xacro="http://www.ros.org/wiki/xacro">
-  <xacro:property name="link_00_name" value="base_link" />
+  <xacro:property name="dummy_link" value="base_link" />
+  <xacro:property name="link_00_name" value="chassis" />
   <xacro:property name="link_01_name" value="base_arm" />
-  <xacro:property name="link_02_name" value="wheel_left" />
-  <xacro:property name="link_03_name" value="wheel_right" />
-  <!-- <xacro:property name="link_04_name" value="wheel_back_right" />
-  <xacro:property name="link_05_name" value="wheel_back_left" /> -->
+  <xacro:property name="link_02_name" value="wheel_front_left" />
+  <xacro:property name="link_03_name" value="wheel_front_right" />
+  <xacro:property name="link_04_name" value="wheel_back_right" />
+  <xacro:property name="link_05_name" value="wheel_back_left" />
   <xacro:property name="link_06_name" value="arm_1" />
   <xacro:property name="link_07_name" value="arm_2" />
